File: hw/smart-roller-gate-controller/smart-roller-gate-controller.kicad_pcb (KiCad board)
At the start: 2 copper layers, 100 x 75 mm, 16 parts, among them K1 PE014005, K2 PE014005

Commit message: hw: initial placement
Parts:
- removed XP5, XP8: Screw_Terminal_01x02, Connector_Wire:SolderWirePad_1x02_P5.08mm_Drill1.5mm
- added F1: Polyfuse 2.5A, Fuse:Fuse_Bourns_MF-RHT1300, F.Cu at (111.0, 141.0)
- added F2: Polyfuse 0.3A, Fuse:Fuse_Bourns_MF-RHT200, F.Cu at (142.0, 153.0)
- added F3: Polyfuse 0.3A, Fuse:Fuse_Bourns_MF-RHT200, F.Cu at (143.0, 138.0)
- added J1: L, Connector_Wire:SolderWirePad_1x01_Drill1.2mm, F.Cu at (103.0, 163.0)
- added J2: N, Connector_Wire:SolderWirePad_1x01_Drill1.2mm, F.Cu at (103.0, 170.0)
- added J3: L_c, Connector_Wire:SolderWirePad_1x01_Drill1.2mm, F.Cu at (105.0, 151.0)
- added J4: N_c, Connector_Wire:SolderWirePad_1x01_Drill1.2mm, F.Cu at (140.0, 160.0)
- added JP1: Jumper_NC_Dual, Jumper:SolderJumper-3_P1.3mm_Open_RoundedPad1.0x1.5mm, F.Cu at (179.0, 117.0)
- added JP2: Jumper_NC_Dual, Jumper:SolderJumper-3_P1.3mm_Open_RoundedPad1.0x1.5mm, F.Cu at (176.0, 117.0)
- added R1: n/c, Resistor_SMD:R_0603_1608Metric_Pad1.05x0.95mm_HandSolder, F.Cu at (144.1, 84.4)
- added R10: 4.7k, Resistor_SMD:R_0603_1608Metric_Pad1.05x0.95mm_HandSolder, F.Cu at (174.4, 128.1)
- added R2: n/c, Resistor_SMD:R_0603_1608Metric_Pad1.05x0.95mm_HandSolder, F.Cu at (157.0, 80.6)
- added R3: 10k, Resistor_SMD:R_0603_1608Metric_Pad1.05x0.95mm_HandSolder, F.Cu at (122.1, 93.0)
- added R4: 4.7k, Resistor_SMD:R_0603_1608Metric_Pad1.05x0.95mm_HandSolder, F.Cu at (144.1, 81.9)
- added R5: 10k, Resistor_SMD:R_0603_1608Metric_Pad1.05x0.95mm_HandSolder, F.Cu at (112.1, 90.0)
- added R6: n/c, Resistor_SMD:R_0603_1608Metric_Pad1.05x0.95mm_HandSolder, F.Cu at (195.2, 86.9)
- added R7: 10k, Resistor_SMD:R_0603_1608Metric_Pad1.05x0.95mm_HandSolder, F.Cu at (123.0, 129.0)
- added R8: 10k, Resistor_SMD:R_0603_1608Metric_Pad1.05x0.95mm_HandSolder, F.Cu at (136.0, 129.0)
- added R9: 4.7k, Resistor_SMD:R_0603_1608Metric_Pad1.05x0.95mm_HandSolder, F.Cu at (178.8, 129.6)
- added RV1: 440V, Varistor:RV_Disc_D21.5mm_W4.9mm_P10mm, F.Cu at (150.0, 140.0)
- added VD1: D, Diode_SMD:D_SOD-123, F.Cu at (118.0, 133.0)
- added VD2: D, Diode_SMD:D_SOD-123, F.Cu at (131.0, 133.0)
- added XP10: FENCE SENSOR POWER, smart-roller-gate-controller:CONN-KF250-BA-4, F.Cu at (150.0, 167.5)
- added XP11: FENCE INPUTS, smart-roller-gate-controller:CONN-KF250-BA-4, F.Cu at (167.5, 167.5)
- added XP4: ROLLER SENSOR, smart-roller-gate-controller:CONN-KF250-BA-4, F.Cu at (185.0, 167.5)
- added XP6: MAINS, smart-roller-gate-controller:CONN-KF250-BA-4, F.Cu at (115.0, 167.5)
- added XP9: ROLLER MOTOR, smart-roller-gate-controller:CONN-KF250-BA-4, F.Cu at (132.5, 167.5)
- moved XP1 170.1 mm to (113.0, 100.5), turned to 180 degrees
- moved XP3 163.4 mm to (111.0, 120.0)
- moved DD2 149.7 mm to (136.0, 110.0)
- moved VT2 146.6 mm to (136.0, 132.0), turned to 270 degrees
- moved VT1 139.3 mm to (123.0, 132.0), turned to 270 degrees
- moved XP2 123.8 mm to (111.0, 112.0)
- moved K2 116.8 mm to (129.0, 136.0), turned to 270 degrees
- moved K1 107.7 mm to (116.0, 136.0), turned to 270 degrees
- moved DD1 103.7 mm to (164.0, 106.0)
- moved XP7 93.1 mm to (184.0, 108.0)
- moved DA1 91.5 mm to (192.7, 145.0)
- moved PS1 73.5 mm to (155.0, 142.5)
- moved C1 53.5 mm to (193.0, 140.0), turned to 180 degrees
- moved C2 31.5 mm to (193.0, 150.0)
Connections:
- DD1 pad 13: (no net) -> /CC_CFG0
- DD1 pad 5: (no net) -> /CC_CFG1
- DD2 pad 6: (no net) -> BLK2
- DD2 pad 7: (no net) -> ~RSNS
- DD2 pad 9: (no net) -> BLK1
- K1 pad 11: (no net) -> /L_m
- K1 pad 14: (no net) -> /L_m2
- K2 pad 14: (no net) -> /L_m1
- PS1 pad 1: (no net) -> /L_sp

Commit message: hw: done initial placement
Parts:
- moved R6 77.2 mm to (127.0, 123.0)
- moved R4 61.0 mm to (179.0, 132.0), turned to 180 degrees
- moved R2 44.4 mm to (144.0, 123.0), turned to 180 degrees
- moved R1 42.5 mm to (107.0, 105.0)
- moved R5 38.0 mm to (127.0, 125.0)
- moved R3 18.1 mm to (107.0, 103.0)
- moved F1 10.8 mm to (107.0, 151.0), turned to 90 degrees
- moved F2 10.3 mm to (147.0, 144.0), turned to 180 degrees
- moved J3 10.2 mm to (103.0, 141.0)
- moved J4 9.90 mm to (147.0, 153.0)
- moved JP1 7.07 mm to (186.0, 118.0)
- moved JP2 7.07 mm to (183.0, 118.0)
- moved R10 4.57 mm to (179.0, 128.1)
- moved F3 4.47 mm to (147.0, 140.0), turned to 180 degrees
- moved PS1 3.00 mm to (158.0, 142.5)
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Connections:
- K1 pad 14: /L_m2 -> /L_m1
- K2 pad 14: /L_m1 -> /L_m2
- XP9 pad 1: /L_m1 -> Earth_Protective
- XP9 pad 2: /L_m2 -> /L_m1
- XP9 pad 3: /N_c -> /L_m2
- XP9 pad 4: Earth_Protective -> /N_c
Routing:
- added copper zone on B.Cu, net GND
- added copper zone on F.Cu, net GND

Commit message: hw: initial traces
Parts:
- moved R5 9.39 mm to (123.0, 116.5), turned to 270 degrees
- moved R6 1.41 mm to (128.0, 122.0)
- moved R8 1.00 mm to (135.0, 129.0)
- moved VD2 1.00 mm to (130.0, 133.0)
- moved VT2 1.00 mm to (135.0, 132.0)
Routing:
- net GPIO0: track 0.00 -> 58.7 mm, vias 0 -> 2
- net PZ_TX: track 0.00 -> 50.4 mm
- net PZ_RX: track 0.00 -> 48.9 mm
- net ~D_CS: track 0.00 -> 43.7 mm, vias 0 -> 2
- net ~S2_CS: track 0.00 -> 42.7 mm
- net +3V3: track 0.00 -> 42.0 mm
- net ESP_RX: track 0.00 -> 35.0 mm, vias 0 -> 1
- net ESP_TX: track 0.00 -> 34.8 mm, vias 0 -> 1
- net GPIO2: track 0.00 -> 34.6 mm
- net /CC_CFG0: track 0.00 -> 34.5 mm
- net /GPIO4: track 0.00 -> 32.7 mm
- net SCK: track 0.00 -> 31.3 mm
- net /~CC_RST: track 0.00 -> 29.4 mm, vias 0 -> 2
- net /CC_CFG1: track 0.00 -> 28.8 mm
- net MOSI: track 0.00 -> 28.6 mm, vias 0 -> 1
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Other:
- net class LV Power added: clearance 0.2, trace_width 0.25, via_dia 0.8, via_drill 0.4
- net class Signal Small added: clearance 0.15, trace_width 0.2, via_dia 0.8, via_drill 0.4
- rule trace_min: 0.2 -> 0.15

Commit message: hw: done v1.0
Parts:
- added G***: LOGO, ninoslavb-footprinti:high, B.Cu at (166.5, 144.5)
- added G***: LOGO, ninoslavb-footprinti:high, F.Cu at (143.5, 131.0)
- added REF**: OSHW-Logo2_9.8x8mm_SilkScreen, Symbol:OSHW-Logo2_9.8x8mm_SilkScreen, F.Cu at (193.5, 120.0)
- J3: value L_c -> L
- J4: value N_c -> N
- JP1: value Jumper_NC_Dual -> CFG0
- JP2: value Jumper_NC_Dual -> CFG1
- XP10: value FENCE SENSOR POWER -> FENCE POWER
- XP7: value Conn_01x04 -> PZEM
- moved R2 40.6 mm to (107.0, 106.2), turned to 0 degrees
- moved F2 7.50 mm to (141.0, 148.5), turned to 90 degrees
- moved R10 0.94 mm to (179.0, 129.0)
- moved R9 0.50 mm to (179.0, 130.5)
- moved R1 0.30 mm to (107.0, 104.7)
Routing:
- net +3V3: track 42.0 -> 252.6 mm, vias 0 -> 4
- net +5V: track 16.9 -> 178.1 mm
- net BLK1: track 0.00 -> 114.6 mm, vias 0 -> 2
- net BLK2: track 0.00 -> 110.3 mm, vias 0 -> 2
- net ~RSNS: track 0.00 -> 102.3 mm, vias 0 -> 2
- net /N_c: track 0.00 -> 54.6 mm
- net GPIO2: track 34.6 -> 81.9 mm, vias 0 -> 2
- net /L_c: track 0.00 -> 45.1 mm
- net /L_m1: track 0.00 -> 29.7 mm
- net Earth_Protective: track 0.00 -> 26.2 mm
- net /L_sens: track 0.00 -> 24.6 mm
- net GND: track 7.95 -> 29.5 mm, vias 0 -> 13
- net /L_lock1_2: track 0.00 -> 13.7 mm
- net /L_m2: track 0.00 -> 13.3 mm
- net /L_sp: track 0.00 -> 12.0 mm
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- added copper zone on F.Cu, net Earth_Protective
Other:
- net class HV Power added: clearance 2, trace_width 1, via_dia 1.2, via_drill 0.7
- net class LV Power: trace_width 0.25 -> 0.5
- board text added: "3V R T G"
- board text added: "5V ~SN~ G G"
- board text added: "L L N N"
- board text added: "L N PE PE"
- board text added: "PE L1 L2 N"
- board text added: "Roller Gate Controller V1.0 (c) 2020 Vladimir Ermakov"
- board text added: "~B1~ G ~B2~ G"
